File: PCB/processing.kicad_sch (KiCad schematic)
At the start: 56 parts, among them J2 AudioJack3, U4 OPA1679, U5 OPA1679, U6 SSI2164, U7 LM331N

Commit message: forgot to push the new theremin duh
Parts:
- removed C27: 100n, Capacitor_SMD:C_0805_2012Metric, symbol Device:C
- removed C28: 10u, Capacitor_SMD:C_0805_2012Metric, symbol Device:C
- removed C31: 1.2n, Capacitor_SMD:C_0805_2012Metric, symbol Device:C
- removed R20: 220, Resistor_SMD:R_0805_2012Metric, symbol Device:R
- removed U6: SSI2164, Package_SO:SOIC-16_3.9x9.9mm_P1.27mm, symbol Audio:SSI2164
- added C35: 100n, Capacitor_SMD:C_0805_2012Metric, symbol Device:C
- added JP1: SolderJumper_3_Open, Jumper:SolderJumper-3_P1.3mm_Open_Pad1.0x1.5mm_NumberLabels, symbol Jumper:SolderJumper_3_Open
- added R12, R15, R24, R30: 100k, Resistor_SMD:R_0805_2012Metric, symbol Device:R
- added R16, R28, R29: 470, Resistor_SMD:R_0805_2012Metric, symbol Device:R
- added R18: 33k, Resistor_SMD:R_0805_2012Metric, symbol Device:R
- added R21: 1M, Resistor_SMD:R_0805_2012Metric, symbol Device:R
- added R23: 1k, Resistor_SMD:R_0805_2012Metric, symbol Device:R
- added R27: 10k, Resistor_SMD:R_0805_2012Metric, symbol Device:R
- added RV1: 50k, Potentiometer_SMD:Potentiometer_Bourns_3224W_Vertical, symbol Device:R_Potentiometer
- added U6: LM13700, Package_SO:SOIC-16_4.55x10.3mm_P1.27mm, symbol Amplifier_Operational:LM13700
- R17: value 20k -> 470
- renumbered C18 to C17, C17 to C18, C21 to C20, C22 to C21, C24 to C22, C25 to C23, C20 to C24, C23 to C25, C29 to C27, C30 to C28, C32 to C29, C33 to C30, C34 to C31, C35 to C32, C36 to C33, C37 to C34, R12 to R13, R13 to R14, R14 to R19, R15 to R20, R16 to R22, R18 to R25, R19 to R26, R21 to R31, R22 to R32, R23 to R33, R24 to R34, R25 to R35, R26 to R36, R27 to R37, RV1 to RV2, RV2 to RV3
Connections:
- net ANA_REF: now also R17.1, R16.1, R18.1, R28.1, R29.1, R30.1
- net ANA_VDD: now also C35.1, R21.2, RV1.1, U6.11 (V+)
- net GND: now also C35.2, R27.1, RV1.3, U6.6 (V-)
- net SEL1: now also R24.1
- net VOL_CV: now also R15.2
- net at C24.1, R19.1, U5.2 (-): now also R23.2
- net at R17.2: now also U6.13 (-)
- new net: R29.2, U6.4 (-)
- new net: JP1.2 (C), R21.1, R30.2, U6.5
- new net: R24.2, R28.2, U6.3 (+)
- new net: U6.1, U6.12
- new net: R18.2, U6.16
- new net: R12.1, R15.1, R16.2, U6.14 (+)
- new net: R12.2, RV1.2
- new net: JP1.3 (B), R23.1, R27.2, U6.9
- new net: JP1.1 (A), U6.10
- no-connect marks 0 -> 6
Other:
- note added: "(optional jumper to short out darlington)"
- note added: "simple output effects with pads for custom RC combinations"
- note removed: "will be a good idea to have a debug output that is not modulated by the volumecontrol"
- moved on the sheet: C17, C24, C25, C26, C27, C28, C29, C30, C31, C32, J2, R19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
