File: PCB/theremin.kicad_pcb (KiCad board)
At the start: 2 copper layers, 50 x 100 mm, 108 parts, among them J1 Conn_01x08_Pin, J2 AudioJack3, J3 PWR, U1 4070, U2 40106, U3 4060B, U4 OPA1679, U5 OPA1679, U6 SSI2164, U7 LM331N, U8 LM317_SOT-223, Y1 8MHz

Commit message: forgot to push the new theremin duh
Parts:
- removed the C27 at (97.4, 105.4)
- removed the C28 at (96.0, 95.0)
- removed the C31 at (87.0, 95.0)
- removed the D1 at (102.0, 113.0)
- removed FB1: FerriteBead_Small, Inductor_SMD:L_0805_2012Metric
- removed the R20 at (90.0, 95.0)
- removed the TP12 at (100.0, 102.0)
- added C35: 100n, Capacitor_SMD:C_0805_2012Metric, F.Cu at (97.5, 105.6)
- added JP2: SolderJumper_2_Open, Jumper:SolderJumper-2_P1.3mm_Open_Pad1.0x1.5mm, F.Cu at (84.8, 117.3)
- added R12: 100k, Resistor_SMD:R_0805_2012Metric, F.Cu at (90.0, 95.0)
- added R15: 100k, Resistor_SMD:R_0805_2012Metric, F.Cu at (90.7, 98.1)
- added R16: 470, Resistor_SMD:R_0805_2012Metric, F.Cu at (100.8, 98.3)
- added R18: 33k, Resistor_SMD:R_0805_2012Metric, F.Cu at (84.6, 101.3)
- added R21: 1M, Resistor_SMD:R_0805_2012Metric, F.Cu at (92.6, 108.7)
- added R23: 1k, Resistor_SMD:R_0805_2012Metric, F.Cu at (79.0, 109.4)
- added R24: 100k, Resistor_SMD:R_0805_2012Metric, F.Cu at (88.4, 108.7)
- added R27: 10k, Resistor_SMD:R_0805_2012Metric, F.Cu at (79.0, 111.9)
- added R28: 470, Resistor_SMD:R_0805_2012Metric, F.Cu at (100.8, 100.9)
- added R29: 470, Resistor_SMD:R_0805_2012Metric, F.Cu at (100.8, 103.9)
- added R30: 100k, Resistor_SMD:R_0805_2012Metric, F.Cu at (92.5, 111.5)
- added RV1: 50k, Potentiometer_SMD:Potentiometer_Bourns_3224W_Vertical, F.Cu at (86.3, 94.3)
- JP1: value Jumper_2_Open -> SolderJumper_3_Open; footprint Resistor_SMD:R_0805_2012Metric -> Jumper:SolderJumper-3_P1.3mm_Open_Pad1.0x1.5mm_NumberLabels
- L1, L2: footprint Capacitor_THT:CP_Radial_Tantal_D8.0mm_P5.00mm -> Inductor_SMD:L_Coilcraft_LPS3314
- R17: value 20k -> 470
- R39: renamed from R29; value 10k -> 500
- U6: value SSI2164 -> LM13700; footprint Package_SO:SOIC-16_3.9x9.9mm_P1.27mm -> Package_SO:SOIC-16_4.55x10.3mm_P1.27mm
- moved JP1 15.8 mm to (95.0, 97.7), turned to 0 degrees
- moved C1 11.7 mm to (79.2, 67.2), turned to -90 degrees
- moved C37 8.67 mm to (93.8, 124.8)
- moved R17 7.79 mm to (100.8, 95.3), turned to 180 degrees
- moved C36 6.21 mm to (91.0, 124.8)
- moved C38 6.21 mm to (87.0, 114.8)
- moved C39 6.21 mm to (83.0, 114.8)
- moved R39 6.21 mm to (88.0, 120.8)
- moved R40 6.21 mm to (88.0, 124.8)
- moved U8 6.21 mm to (93.0, 117.8)
- moved C13 4.65 mm to (72.8, 45.8)
- moved C5 4.65 mm to (91.2, 45.8)
- moved D1 2.00 mm to (79.4, 123.0)
- moved J3 2.00 mm to (80.8, 126.0)
- moved R38 2.00 mm to (84.3, 123.0)
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- renumbered C18 to C17, C17 to C18, C21 to C20, C22 to C21, C24 to C22, C25 to C23, C20 to C24, C23 to C25, C29 to C27, C30 to C28, C32 to C29, C33 to C30, C34 to C31, C35 to C32, C36 to C33, C37 to C34, C39 to C36, C40 to C37, C41 to C38, C42 to C39, D2 to D1, R12 to R13, R13 to R14, R14 to R19, R15 to R20, R16 to R22, R18 to R25, R19 to R26, R21 to R31, R22 to R32, R23 to R33, R24 to R34, R25 to R35, R26 to R36, R27 to R37, R28 to R38, R30 to R40, RV1 to RV2, RV2 to RV3, TP13 to TP12
Connections:
- net /Signal Processing/SINE_OUT renamed /Signal Processing/EFFECT_1
- net /Signal Processing/SQUARE_OUT renamed /Signal Processing/EFFECT_2
- net /Signal Processing/TRI_OUT renamed /Signal Processing/EFFECT_3
- JP1 pad 1: Net-(D1-A) (its old number) -> Net-(JP1-A)
- JP1 pad 2: VDD -> Net-(JP1-C)
- R17 pad 1: Net-(C28-Pad2) -> ANA_REF
- R17 pad 2: Net-(U6-I_IN1) -> Net-(U6A--)
- R39 pad 1: Net-(D1-A) (its old number) -> VDD
- U1 pad 14: GND -> VDD
- U1 pad 7: VDD -> GND
- U6 pad 1: unconnected-(U6-MODE-Pad1) -> Net-(U6-Pad1)
- U6 pad 10: unconnected-(U6-I_IN3-Pad10) -> Net-(JP1-A)
- U6 pad 11: unconnected-(U6-VC3-Pad11) -> ANA_VDD
- U6 pad 12: unconnected-(U6-I_OUT3-Pad12) -> Net-(U6-Pad1)
- U6 pad 13: unconnected-(U6-I_OUT4-Pad13) -> Net-(U6A--)
- U6 pad 14: unconnected-(U6-VC4-Pad14) -> Net-(U6A-+)
- U6 pad 16: ANA_VDD -> Net-(R18-Pad2)
- U6 pad 2: Net-(U6-I_IN1) -> unconnected-(U6C-DIODE_BIAS-Pad2)
- U6 pad 3: /Signal Processing/VOL_CV -> Net-(U6C-+)
- U6 pad 4: Net-(U5A--) -> Net-(U6C--)
- U6 pad 5: unconnected-(U6-I_OUT2-Pad5) -> Net-(JP1-C)
- U6 pad 6: unconnected-(U6-VC2-Pad6) -> GND
- U6 pad 8: ANA_REF -> unconnected-(U6-Pad8)
- U6 pad 9: GND -> Net-(JP1-B)
- U8 pad 2: Net-(D1-A) (its old number) -> VDD
Routing:
- net Net-(JP1-B): track 0.00 -> 34.3 mm, vias 0 -> 4
- net ANA_REF: track 111.5 -> 136.6 mm, vias 12 -> 13
- net Net-(JP1-C): track 0.00 -> 24.1 mm, vias 0 -> 2
- net Net-(D1-A) (its old number): track 20.9 -> 0.00 mm
- net Net-(U6A-+): track 0.00 -> 20.3 mm, vias 0 -> 2
- net /Signal Processing/PITCH_FILTERED: track 69.0 -> 88.7 mm
- net Net-(U6C-+): track 0.00 -> 15.7 mm, vias 0 -> 2
- net Net-(U6A--): track 0.00 -> 15.0 mm, vias 0 -> 2
- net Net-(J3-Pin_2): track 52.4 -> 38.1 mm
- net Net-(U6C--): track 0.00 -> 11.2 mm, vias 0 -> 2
- net Net-(U6-Pad1): track 0.00 -> 11.0 mm, vias 0 -> 4
- net /Signal Processing/VOL_CV: track 40.5 -> 30.3 mm
- net Net-(U5A--): track 24.6 -> 15.8 mm
- net Net-(U6-I_IN1): track 8.67 -> 0.00 mm
- net ANA_VDD: track 143.0 -> 150.2 mm
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