File: PCB Legacy/oscillators.kicad_sch (KiCad schematic)
At the start: 31 parts, among them U1 4070, U2 40106, U3 4060B, Y1 8MHz

Commit message: forgot to push the new theremin duh
Parts:
- L1, L2: footprint Inductor_SMD:L_Coilcraft_LPS3314 -> Capacitor_THT:CP_Radial_Tantal_D8.0mm_P5.00mm
Connections:
- net GND: now also U1.14 (VDD); no longer U1.7 (VSS)
- net VDD: now also U1.7 (VSS); no longer U1.14 (VDD)
- no-connect marks 11 -> 1
Other:
- note added: "PITCH f="
- note added: "VOLUME f="
- note added: "make this as large as possible"
- note added: "wow"
- note removed: "PITCH f=500k"
- note removed: "VOLUME f=250k"
- note removed: "spare pad for tuning capacitance (if needed)"
Changed lines of the file:
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@@
 	(generator_version "9.0")
 	(paper "A4")
-	(text "VOLUME f=250k\n\n"
+	(text "wow "
+		(exclude_from_sim no)
+		(at 269.24 121.92 0)
+		(effects
+			(font
+				(size 1.27 1.27)
+				(thickness 0.254)
+				(bold yes)
+			)
+		)
+	)
+	(text "VOLUME f=\n\n\n"
 		(exclude_from_sim no)
 		(at 38.1 105.41 0)
@@
 		)
 	)
-	(text "spare pad for tuning capacitance\n(if needed)"
+	(text "make this as large as possible\n"
 		(exclude_from_sim no)
-		(at 55.88 87.63 0)
+		(at 43.18 87.63 0)
 		(effects
 			(font
@@
 		)
 	)
-	(text "PITCH f=500k\n"
+	(text "PITCH f=\n"
 		(exclude_from_sim no)
 		(at 40.64 40.64 0)
@@
 	)
 	(no_connect
-		(at 208.28 72.39)
-	)
-	(no_connect
-		(at 243.84 25.4)
-	)
-	(no_connect
-		(at 208.28 57.15)
-	)
-	(no_connect
-		(at 208.28 59.69)
-	)
-	(no_connect
-		(at 279.4 25.4)
-	)
-	(no_connect
-		(at 208.28 77.47)
-	)
-	(no_connect
 		(at 182.88 52.07)
 	)
-	(no_connect
-		(at 208.28 64.77)
-	)
-	(no_connect
-		(at 208.28 62.23)
-	)
-	(no_connect
-		(at 208.28 74.93)
-	)
-	(no_connect
-		(at 208.28 67.31)
-	)
 	(wire
 		(pts
@@
 	)
 	(symbol
+		(lib_id "4xxx:4070")
+		(at 252.73 129.54 180)
+		(unit 5)
+		(exclude_from_sim no)
+		(in_bom yes)
+		(on_board yes)
+		(dnp no)
+		(fields_autoplaced yes)
+		(property "Reference" "U1"
+			(at 259.08 128.2699 0)
+			(effects
+				(font
+					(size 1.27 1.27)
+				)
+				(justify right)
+			)
+		)
+		(property "Value" "4070"
+			(at 259.08 130.8099 0)
+			(effects
+				(font
+					(size 1.27 1.27)
+				)
+				(justify right)
+			)
+		)
+		(property "Footprint" "Package_SO:SOIC-14_3.9x8.7mm_P1.27mm"
+			(at 252.73 129.54 0)
+			(effects
+				(font
+					(size 1.27 1.27)
+				)
+				(hide yes)
+			)
+		)
+		(property "Datasheet" "http://www.intersil.com/content/dam/Intersil/documents/cd40/cd4070bms-77bms.pdf"
+			(at 252.73 129.54 0)
+			(effects
+				(font
+					(size 1.27 1.27)
+				)
+				(hide yes)
+			)
+		)
+		(property "Description" "Quad Xor 2 inputs"
+			(at 252.73 129.54 0)
+			(effects
+				(font
+					(size 1.27 1.27)
+				)
+				(hide yes)
+			)
+		)
+		(pin "2"
+		)
+		(pin "3"
+		)
+		(pin "1"
+		)
+		(pin "6"
+		)
+		(pin "4"
+		)
+		(pin "8"
+		)
+		(pin "9"
+		)
+		(pin "10"
+		)
+		(pin "12"
+		)
+		(pin "13"
+		)
+		(pin "11"
+		)
+		(pin "14"
+		)
+		(pin "7"
+		)
+		(pin "5"
+		)
+		(instances
+			(project ""
+				(path "/2ea7cf03-dad6-47d0-8fed-accfb6b9ebf9/5c5df33e-e39a-4938-8e1e-936d5173d3b4"
+					(reference "U1")
+					(unit 5)
+				)
+			)
+		)
+	)
+	(symbol
 		(lib_id "Device:C")
 		(at 86.36 144.78 0)
@@
 			)
 		)
-		(property "Footprint" "Inductor_SMD:L_Coilcraft_LPS3314"
+		(property "Footprint" "Capacitor_THT:CP_Radial_Tantal_D8.0mm_P5.00mm"
 			(at 76.2 63.5 0)
 			(effects
@@
 			)
 		)
-		(property "Footprint" "Inductor_SMD:L_Coilcraft_LPS3314"
+		(property "Footprint" "Capacitor_THT:CP_Radial_Tantal_D8.0mm_P5.00mm"
 			(at 76.2 133.35 0)
 			(effects
@@
 				)
 			)
-		)
-	)
-	(symbol
-		(lib_id "4xxx:4070")
-		(at 252.73 129.54 0)
-		(unit 5)
-		(exclude_from_sim no)
-		(in_bom yes)
-		(on_board yes)
-		(dnp no)
-		(fields_autoplaced yes)
-		(property "Reference" "U1"
-			(at 259.08 128.2699 0)
-			(effects
-				(font
-					(size 1.27 1.27)
-				)
-				(justify left)
-			)
-		)
-		(property "Value" "4070"
-			(at 259.08 130.8099 0)
-			(effects
-				(font
-					(size 1.27 1.27)
-				)
-				(justify left)
-			)
-		)
-		(property "Footprint" "Package_SO:SOIC-14_3.9x8.7mm_P1.27mm"
-			(at 252.73 129.54 0)
-			(effects
-				(font
-					(size 1.27 1.27)
-				)
-				(hide yes)
-			)
-		)
-		(property "Datasheet" "http://www.intersil.com/content/dam/Intersil/documents/cd40/cd4070bms-77bms.pdf"
-			(at 252.73 129.54 0)
-			(effects
-				(font
-					(size 1.27 1.27)
-				)
-				(hide yes)
-			)
-		)
-		(property "Description" "Quad Xor 2 inputs"
-			(at 252.73 129.54 0)
-			(effects
-				(font
-					(size 1.27 1.27)
-				)
-				(hide yes)
-			)
-		)
-		(pin "2"
-		)
-		(pin "3"
-		)
-		(pin "1"
-		)
-		(pin "6"
-		)
-		(pin "4"
-		)
-		(pin "8"
-		)
-		(pin "9"
-		)
-		(pin "10"
-		)
-		(pin "12"
-		)
-		(pin "13"
-		)
-		(pin "11"
-		)
-		(pin "14"
-		)
-		(pin "7"
-		)
-		(pin "5"
-		)
-		(instances
-			(project "theremin"
-				(path "/2ea7cf03-dad6-47d0-8fed-accfb6b9ebf9/5c5df33e-e39a-4938-8e1e-936d5173d3b4"
-					(reference "U1")
-					(unit 5)
-				)
-			)
