File: PCB Legacy/psu.kicad_sch (KiCad schematic)
At the start: 13 parts, among them J3 PWR, U8 LM317_SOT-223

Commit message: forgot to push the new theremin duh
Parts:
- removed JP2: SolderJumper_2_Open, Jumper:SolderJumper-2_P1.3mm_Open_Pad1.0x1.5mm, symbol Jumper:SolderJumper_2_Open
- added D1: 1N4002, Diode_SMD:D_0805_2012Metric, symbol Diode:1N4002
- added FB1: FerriteBead_Small, Inductor_SMD:L_0805_2012Metric, symbol Device:FerriteBead_Small
- added JP1: Jumper_2_Open, Resistor_SMD:R_0805_2012Metric, symbol Jumper:Jumper_2_Open
- added TP12: VDD_ANA, TestPoint:TestPoint_Pad_2.0x2.0mm, symbol Connector:TestPoint
- C40: renamed from C37; value 100n -> 100u
- R29: renamed from R39; value 240 -> 10k
- R30: renamed from R40; value 2k -> 1.2k
- renumbered C36 to C39, C38 to C41, C39 to C42, D1 to D2, R38 to R28, TP12 to TP13
Connections:
- net ANA_VDD: now also FB1.2, TP12.1
- net VDD: now also FB1.1, JP1.2 (B); no longer R29.1, U8.2 (VO)
- net at C39.1, C40.1, J3.2 (Pin_2)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: now also D1.1 (K)
- new net: D1.2 (A), JP1.1 (A), R29.1, U8.2 (VO)
Other:
- note added: "give this an 0805 footprint"
- note added: "incorrect value"
- note removed: "short this jumper"
- note removed: "~10-12V"
- moved on the sheet: C39, C40, C41, C42, D2, J3, R28, R29, R30, TP11, TP13, U8
